Commit message: Added elbow and shoulder along w collision for model

File: collision_detection/urdf/project_arm.urdf (robot description, URDF)
Before this commit: robot side_mount_arm_2link, 4 links, 3 joints
Links:
- link base_link: geometry collision cylinder length=0.10 radius=0.095; visual cylinder length=0.10 radius=0.10
- link link0: geometry collision cylinder length=0.10 radius=0.09; visual cylinder length=0.10 radius=0.10
- link link1: geometry collision cylinder length=0.35 radius=0.045; collision sphere radius=0.08
- link link2: geometry collision cylinder length=0.35 radius=0.045; collision sphere radius=0.08
Joints:
- joint base_yaw: origin xyz=0 0 0.10 -> xyz=0 0 0.155
- joint elbow_hinge: origin xyz=-0.15 0 0.35 -> xyz=-0.18 0 0.35
- joint side_hinge: origin xyz=0.15 0 0.05 -> xyz=0.22 0 0.05
