Commit message: Final Commit for the Sem. Goodbye

File: robot_driver/urdf/project_arm.urdf (robot description, URDF)
Before this commit: robot side_mount_arm_2link_clean, 4 links, 3 joints
Links:
- added link link3; collision cylinder length=0.1 radius=0.0225; collision sphere radius=0.04
Joints:
- added joint node3: type revolute, parent link2, child link3, origin xyz=0 0 0.35, axis -1 0 0, limit lower=-3.1416 upper=3.1416 effort=10 velocity=2
